Commit message: The bulldozer d37pxi in the AGX Simulator can be controlled by nav2.

File: d37pxi_description/urdf/d37pxi24.xacro (robot description, xacro)
@@ -5,13 +5,14 @@
 <!-- =================================================================================== -->
 <!-- <xacro:property name="robot_name" value="d37pxi24" /> -->
-<robot xmlns:xacro="http://www.ros.org/wiki/xacro" name="d37pxi24">
+<robot xmlns:xacro="http://www.ros.org/wiki/xacro" name="d37pxi">
+  <xacro:property name="tf_prefix" value=""/>
   <!-- Base Link -->
-  <link name="base_link"/>
+  <link name="${tf_prefix}/base_link"/>
   <!-- Body {{{ -->
   <joint name="base_joint" type="fixed">
-    <parent link="base_link"/>
-    <child link="body_link"/>
-  </joint>
-  <link name="body_link">
+    <parent link="${tf_prefix}/base_link"/>
+    <child link="${tf_prefix}/body_link"/>
+  </joint>
+  <link name="${tf_prefix}/body_link">
     <visual>
       <geometry>
@@ -32,12 +33,12 @@
   <!-- }}} Body ends here -->
   <!-- Blade Arm {{{ -->
-  <joint name="blade_arm_joint" type="revolute">
+  <joint name="lift_joint" type="revolute">
     <origin xyz="0.6718 0 0.38606"/>
     <axis xyz="0 1 0"/>
-    <parent link="body_link"/>
-    <child link="blade_arm_link"/>
+    <parent link="${tf_prefix}/body_link"/>
+    <child link="${tf_prefix}/blade_arm_link"/>
     <limit effort="500" lower="-0.41015237421866746" upper="0.18675022996339324" velocity="6.159937255"/>
   </joint>
-  <link name="blade_arm_link">
+  <link name="${tf_prefix}/blade_arm_link">
     <visual>
       <origin xyz="0 0 0"/>
@@ -63,9 +64,9 @@
     <origin xyz="0.54437 0 0.90368"/>
     <axis xyz="0 1 0"/>
-    <parent link="body_link"/>
-    <child link="blade_arm_cylinder_link"/>
-    <mimic joint="blade_arm_joint" multiplier="0.9"/>
-  </joint>
-  <link name="blade_arm_cylinder_link">
+    <parent link="${tf_prefix}/body_link"/>
+    <child link="${tf_prefix}/blade_arm_cylinder_link"/>
+    <mimic joint="lift_joint" multiplier="0.9"/>
+  </joint>
+  <link name="${tf_prefix}/blade_arm_cylinder_link">
     <visual>
       <origin xyz="0 0 0"/>
@@ -91,10 +92,10 @@
     <origin xyz="0 0 0"/>
     <axis xyz="1.0055 0 -0.056785"/>
-    <parent link="blade_arm_cylinder_link"/>
-    <child link="blade_arm_piston_link"/>
+    <parent link="${tf_prefix}/blade_arm_cylinder_link"/>
+    <child link="${tf_prefix}/blade_arm_piston_link"/>
     <limit effort="500" lower="-0.22" upper="0.05" velocity="6.159937255"/>
     <mimic joint="blade_arm_cylinder_joint" multiplier="0.6"/>
   </joint>
-  <link name="blade_arm_piston_link">
+  <link name="${tf_prefix}/blade_arm_piston_link">
     <visual>
       <origin xyz="0 0 0"/>
@@ -117,12 +118,12 @@
   <!-- }}} Blade Arm Piston ends here -->
   <!-- Blade Angle {{{ -->
-  <joint name="blade_angle_joint" type="revolute">
+  <joint name="angle_joint" type="revolute">
     <origin xyz="1.5881 0 -0.10373"/>
     <axis xyz="0 0 1"/>
-    <parent link="blade_arm_link"/>
-    <child link="blade_angle_link"/>
+    <parent link="${tf_prefix}/blade_arm_link"/>
+    <child link="${tf_prefix}/blade_angle_link"/>
     <limit effort="500" lower="-0.4188790204786391" upper="0.4188790204786391" velocity="6.159937255"/>
   </joint>
-  <link name="blade_angle_link"/>
+  <link name="${tf_prefix}/blade_angle_link"/>
   <!-- }}} Blade Angle ends here -->
   <!-- Blade Angle Piston Right {{{ -->
@@ -130,10 +131,10 @@
     <origin xyz="0.50775 -0.44941 0.18324"/>
     <axis xyz="1.093 -0.059226 -0.062315"/>
-    <parent link="blade_arm_link"/>
-    <child link="blade_angle_piston_right_link"/>
+    <parent link="${tf_prefix}/blade_arm_link"/>
+    <child link="${tf_prefix}/blade_angle_piston_right_link"/>
     <limit effort="500" lower="-0.24" upper="0.18" velocity="6.159937255"/>
-    <mimic joint="blade_angle_joint" multiplier="0.5"/>
-  </joint>
-  <link name="blade_angle_piston_right_link">
+    <mimic joint="angle_joint" multiplier="0.5"/>
+  </joint>
+  <link name="${tf_prefix}/blade_angle_piston_right_link">
     <visual>
       <origin xyz="0 0 0"/>
@@ -159,10 +160,10 @@
     <origin xyz="0.50775 0.44941 0.18324"/>
     <axis xyz="1.093 0.059226 -0.062315"/>
-    <parent link="blade_arm_link"/>
-    <child link="blade_angle_piston_left_link"/>
+    <parent link="${tf_prefix}/blade_arm_link"/>
+    <child link="${tf_prefix}/blade_angle_piston_left_link"/>
     <limit effort="500" lower="-0.24" upper="0.18" velocity="6.159937255"/>
-    <mimic joint="blade_angle_joint" multiplier="-0.5"/>
-  </joint>
-  <link name="blade_angle_piston_left_link">
+    <mimic joint="angle_joint" multiplier="-0.5"/>
+  </joint>
+  <link name="${tf_prefix}/blade_angle_piston_left_link">
     <visual>
       <origin xyz="0 0 0"/>
@@ -185,12 +186,12 @@
   <!-- }}} Blade Angle Piston Left ends here -->
   <!-- Blade Tilt {{{ -->
-  <joint name="blade_tilt_joint" type="revolute">
+  <joint name="tilt_joint" type="revolute">
     <origin xyz="0 0 0"/>
     <axis xyz="1 0 0"/>
-    <parent link="blade_angle_link"/>
-    <child link="blade_link"/>
+    <parent link="${tf_prefix}/blade_angle_link"/>
+    <child link="${tf_prefix}/blade_link"/>
     <limit effort="500" lower="-0.1363596851440582" upper="0.1363596851440582" velocity="6.159937255"/>
   </joint>
-  <link name="blade_link">
+  <link name="${tf_prefix}/blade_link">
     <visual>
       <origin xyz="0 0 0"/>

Commit message: Add GNSS link in urdf model (temporary)

File: d37pxi_description/urdf/d37pxi24.xacro (robot description, xacro)
@@ -11,4 +11,6 @@
   <!-- Body {{{ -->
   <joint name="base_joint" type="fixed">
+    <!-- 暫定値 -->
+    <origin xyz="-0.086289 0 0"/>
     <parent link="${tf_prefix}/base_link"/>
     <child link="${tf_prefix}/body_link"/>
@@ -31,4 +33,13 @@
     </inertial>
   </link>
+  <!-- GNSS (Hemisphere V500) {{{ -->
+  <joint name="gnss_temp_joint" type="fixed">
+    <!-- 暫定値 -->
+    <!-- <origin xyz="0.335772 -0.285 2.945"/>     -->
+    <origin xyz="0.335772 -0.285 0"/>  <!-- without height -->
+    <parent link="${tf_prefix}/body_link"/>
+    <child link="${tf_prefix}/gnss_temp_link"/>
+  </joint>
+  <link name="${tf_prefix}/gnss_temp_link"/>
   <!-- }}} Body ends here -->
   <!-- Blade Arm {{{ -->

Commit message: for cmd_vel_control

File: d37pxi_description/urdf/d37pxi24.xacro (robot description, xacro)
@@ -37,5 +37,8 @@
     <!-- 暫定値 -->
     <!-- <origin xyz="0.335772 -0.285 2.945"/>     -->
-    <origin xyz="0.335772 -0.285 0"/>  <!-- without height -->
+    <!-- without height -->
+    <!-- <origin xyz="0.335772 -0.285 0"/>  -->
+    <!-- without height 251111_new_position-->
+    <origin xyz="0.185772 -0.285 0"/>
     <parent link="${tf_prefix}/body_link"/>
     <child link="${tf_prefix}/gnss_temp_link"/>

Commit message: Update: d37pix_unity, navigation周りのプログラムを整備

File: d37pxi_description/urdf/d37pxi24.xacro (robot description, xacro)
@@ -6,5 +6,6 @@
 <!-- <xacro:property name="robot_name" value="d37pxi24" /> -->
 <robot xmlns:xacro="http://www.ros.org/wiki/xacro" name="d37pxi">
-  <xacro:property name="tf_prefix" value=""/>
+  <xacro:arg name="tf_prefix" default=""/>
+  <xacro:property name="tf_prefix" value="$(arg tf_prefix)"/>
   <!-- Base Link -->
   <link name="${tf_prefix}/base_link"/>

Commit message: Setting Nav2 params in the note PC

File: d37pxi_description/urdf/d37pxi24.xacro (robot description, xacro)
@@ -34,15 +34,17 @@
   </link>
   <!-- GNSS (Hemisphere V500) {{{ -->
-  <joint name="gnss_temp_joint" type="fixed">
-    <!-- 暫定値 -->
-    <!-- <origin xyz="0.335772 -0.285 2.945"/>     -->
-    <!-- without height -->
-    <!-- <origin xyz="0.335772 -0.285 0"/>  -->
-    <!-- without height 251111_new_position-->
+  <!-- <joint name="gnss_temp_joint" type="fixed">
     <origin xyz="0.185772 -0.285 0"/>
     <parent link="${tf_prefix}/body_link"/>
     <child link="${tf_prefix}/gnss_temp_link"/>
   </joint>
-  <link name="${tf_prefix}/gnss_temp_link"/>
+  <link name="${tf_prefix}/gnss_temp_link"/> -->
+  <!-- GNSS (Septentrio GNSS) {{{ -->
+  <!-- <joint name="gnss_temp_joint" type="fixed">
+    <origin xyz="0.185772 -0.285 0"/>
+    <parent link="${tf_prefix}/body_link"/>
+    <child link="${tf_prefix}/gnss_temp_link"/>
+  </joint>
+  <link name="${tf_prefix}/gnss_temp_link"/> -->
   <!-- }}} Body ends here -->
   <!-- Blade Arm {{{ -->
